Commit message: completed detector

File: urdf/robot_assignment.xacro (robot description, xacro)
@@ -4,22 +4,20 @@
     <xacro:include filename="$(find ExpRoLab_Assignment2)/urdf/robot_assignment.gazebo" />
     <!-- Macros for inertia -->
-    <xacro:macro name="default_inertial" params="mass">
-        <inertial>
-            <mass value="${mass}" />
-                <origin rpy="0 1.5707 1.5707" xyz="0 0 0"/>
-                <inertia ixx="0.000526666666667" ixy="0" ixz="0" iyy="0.000526666666667" iyz="0" izz="0.001"/>
-        </inertial>
-    </xacro:macro>
     <xacro:macro name="cylinder_inertia" params="mass r l">
-        <inertia ixx="${mass*(3*r*r+l*l)/12}" ixy = "0" ixz = "0" iyy="${mass*(3*r*r+l*l)/12}" iyz = "0" izz="${mass*(r*r)/2}" />
+        <inertia ixx="${mass*(3*r*r+l*l)/12}" ixy = "0" ixz = "0"
+                 iyy="${mass*(3*r*r+l*l)/12}" iyz = "0" izz="${mass*(r*r)/2}" />
+    </xacro:macro>
+    <xacro:macro name="box_inertia" params="x y z mass">
+        <inertia ixx="${mass*(y*y+z*z)/12}" ixy="0.0" ixz="0.0"
+                 iyy="${mass*(x*x+z*z)/12}" iyz="0.0" izz="${mass*(x*x+y*y)/12}" />
     </xacro:macro>
     <!-- Macros with relative properties for the geometry -->
     <xacro:property name="wheel_length" value="0.04" />
-    <xacro:property name="wheel_radius" value="0.08" />
+    <xacro:property name="wheel_radius" value="0.1" />
     <xacro:macro name="wheel_geometry">
         <geometry>
             <cylinder length="${wheel_length}" radius="${wheel_radius}"/>
         </geometry>
-        </xacro:macro>
+    </xacro:macro>
     <xacro:property name="arm_link_length" value="0.15" />
     <xacro:property name="arm_link_radius" value="0.05" />
@@ -35,17 +33,14 @@
                 <mass value="0.2"/>
                 <origin rpy="0 1.5707 1.5707" xyz="0 0 0"/>
-                <inertia ixx="0.000526666666667" ixy="0" ixz="0" iyy="0.000526666666667" iyz="0" izz="0.001"/>
+                <xacro:cylinder_inertia mass="0.2" r="${wheel_radius}" l="${wheel_length}"/>
             </inertial>
-            <collision name="link_right_wheel_collision">
+            <collision name="${name}_collision">
                 <origin rpy="0 1.5707 1.5707" xyz="0 0 0"/>
-                <geometry>
-                    <cylinder length="0.04" radius="0.1"/>
-                </geometry>
+                <xacro:wheel_geometry />
             </collision>
             <visual name="${name}_visual">
                 <origin rpy="0 1.5707 1.5707" xyz="0 0 0"/>
-                <geometry>
-                    <cylinder length="0.04" radius="0.1"/>
-                </geometry>
+                <xacro:wheel_geometry />
+                <material name="blue"/>
             </visual>
         </link>
@@ -57,5 +52,5 @@
                 <mass value="0.025"/>
                 <origin xyz="0 0 0" rpy="0 0 0"/>
-                <xacro:cylinder_inertia mass="0.025" r="0.05" l="0.15"/>
+                <xacro:cylinder_inertia mass="0.025" r="${arm_link_radius}" l="${arm_link_length}"/>
             </inertial>
             <collision name="${name}_collision">
@@ -66,4 +61,5 @@
                 <origin rpy="0 0 0" xyz="0 0 0.075"/>
                 <xacro:arm_link_geometry />
+                <material name="red"/>
             </visual>
         </link>
@@ -75,26 +71,33 @@
         <child link="${child}"/>
         <parent link="${parent}"/>
-        <axis rpy="0 0 0" xyz="0 1 0"/>
-        <limit effort="10000" velocity="1000"/>
+        <axis rpy="0 0 0" xyz="${axis_xyz}"/>
+        <limit effort="10" velocity="10"/>
         <joint_properties damping="1.0" friction="1.0"/>
         </joint>
     </xacro:macro>
-    <xacro:macro name="revolute_joint" params="name child parent origin_xyz">
+    <xacro:macro name="revolute_joint" params="name child parent origin_xyz axis_xyz">
         <joint name="${name}" type="revolute">
             <origin rpy="0 0 0" xyz="${origin_xyz}"/>
             <child link="${child}"/>
             <parent link="${parent}"/>
-            <axis rpy="0 0 0" xyz="1 0 0"/>
-            <limit effort="100.0" upper = "1.5" lower = "-1.5" velocity="0.5"/>
-            <joint_properties damping="1.0" friction="1.0"/>
+            <axis rpy="0 0 0" xyz="${axis_xyz}"/>
+            <limit effort="10.0" upper = "1.0" lower = "-1.0" velocity="0.5"/>
+            <joint_properties damping="10.0" friction="0.1"/>
         </joint>
     </xacro:macro>
+    <xacro:macro name="fixed_joint" params="name child parent origin_xyz">
+        <joint name="${name}" type="fixed">
+            <origin rpy="0 0 0" xyz="${origin_xyz}"/>
+            <child link="${child}"/>
+            <parent link="${parent}"/>
+        </joint>
+    </xacro:macro>
     <!-- Create the chassis of the robot -->
-    <link name="chassis_link">
+    <link name="link_chassis">
         <pose>0 0 0.1 0 0 0</pose>
         <inertial>
             <mass value="5"/>
             <origin rpy="0 0 0" xyz="0 0 0.1"/>
-            <inertia ixx="0.0395416666667" ixy="0" ixz="0" iyy="0.106208333333" iyz="0" izz="0.106208333333"/>
+            <xacro:box_inertia mass="5" x="0.5" y="0.3" z="0.07"/>
         </inertial>
         <collision name="collision_chassis">
@@ -108,5 +111,5 @@
                 <box size="0.5 0.3 0.07"/>
             </geometry>
-            <material name="blue"/>
+            <material name="orange"/>
         </visual>
         <!-- Caster front -->
@@ -137,6 +140,6 @@
     <xacro:link_wheel name="link_right_wheel" />
     <xacro:link_wheel name="link_left_wheel" />
-    <xacro:continuous_joint name="joint_right_wheel" child="link_right_wheel" parent="chassis_link" origin_xyz="-0.05 0.15 0" axis_xyz="0 1 0"/>
-    <xacro:continuous_joint name="joint_left_wheel" child="link_left_wheel" parent="chassis_link" origin_xyz="-0.05 -0.15 0" axis_xyz="0 1 0"/>
+    <xacro:continuous_joint name="joint_right_wheel" child="link_right_wheel" parent="link_chassis" origin_xyz="-0.05 0.15 0" axis_xyz="0 1 0"/>
+    <xacro:continuous_joint name="joint_left_wheel" child="link_left_wheel" parent="link_chassis" origin_xyz="-0.05 -0.15 0" axis_xyz="0 1 0"/>
     <!-- Create the arm base link and its joint -->
     <link name="arm_base_link">
@@ -144,5 +147,5 @@
             <mass value="0.2"/>
             <origin xyz="0 0 0" rpy="0 0 0" />
-            <inertia ixx="0.000208333333333" ixy="0" ixz="0" iyy="0.000208333333333" iyz="0" izz="0.008333333333333"/>
+            <xacro:box_inertia mass="0.2" x="0.1" y="0.1" z="0.05"/>
         </inertial>
         <collision>
@@ -160,12 +163,12 @@
         </visual>
     </link>
-    <xacro:continuous_joint name="arm_base_joint" child="arm_base_link" parent="chassis_link" origin_xyz="0 0 0.06" axis_xyz="0 0 1"/>
+    <xacro:fixed_joint name="arm_base_joint" child="arm_base_link" parent="link_chassis" origin_xyz="0 0 0.06" />
     <!-- Create the arm link and their joints -->
     <xacro:arm_link name="arm_link_01"/>
 	<xacro:arm_link name="arm_link_02"/>
 	<xacro:arm_link name="arm_link_03"/>
-    <xacro:revolute_joint name="arm_joint_01" child="arm_link_01" parent="arm_base_link" origin_xyz="0 0 0.025"/>
-	<xacro:revolute_joint name="arm_joint_02" child="arm_link_02" parent="arm_link_01" origin_xyz="0 0 0.15"/>
-	<xacro:revolute_joint name="arm_joint_03" child="arm_link_03" parent="arm_link_02" origin_xyz="0 0 0.15"/>
+    <xacro:continuous_joint name="arm_joint_01" child="arm_link_01" parent="arm_base_link" origin_xyz="0 0 0.025" axis_xyz="0 0 1"/>
+	<xacro:revolute_joint name="arm_joint_02" child="arm_link_02" parent="arm_link_01" origin_xyz="0 0 0.15" axis_xyz="0 1 0"/>
+	<xacro:revolute_joint name="arm_joint_03" child="arm_link_03" parent="arm_link_02" origin_xyz="0 0 0.15" axis_xyz="0 1 0"/>
     <!-- Create the camera -->
     <link name="camera_link">
@@ -173,5 +176,5 @@
             <mass value="1e-5" />
             <origin xyz="0 0 0" rpy="0 0 0"/>
-            <inertia ixx="1e-6" ixy="0" ixz="0" iyy="1e-6" iyz="0" izz="1e-6" />
+            <xacro:box_inertia mass="1e-5" x="0.1" y="0.1" z="0.1"/>
         </inertial>
         <collision>
@@ -186,15 +189,7 @@
                 <box size="0.1 0.1 0.1"/>
             </geometry>
-            <material name="blue">
-                <color rgba="1 0 0 1"/>
-            </material>
         </visual>
 	</link>
-    <joint name="camera_joint" type="fixed">
-        <axis xyz="0 1 0"/>
-        <origin xyz="0 0 0.15" rpy="0 0 0"/>
-        <parent link="arm_link_03"/>
-        <child link="camera_link"/>
-    </joint>
+    <xacro:fixed_joint name="camera_joint" child="camera_link" parent="arm_link_03" origin_xyz="0 0 0.15" />
     <!-- Create the laser -->
     <link name="laser">
@@ -218,13 +213,9 @@
         </collision>
     </link>
-    <joint name="joint_laser" type="fixed">
-        <origin xyz="0.15 0 0.05" rpy="0 0 0"/>
-        <parent link="chassis_link"/>
-        <child link="laser"/>
-    </joint>
+    <xacro:fixed_joint name="laser_joint" child="laser" parent="link_chassis" origin_xyz="0.15 0 0.05" />
     <!-- Define the transmissions -->
-	<transmission name="arm_base_joint_trans">
+	<transmission name="arm_joint_01_trans">
 		<type>transmission_interface/SimpleTransmission</type>
-		<joint name="arm_base_joint">
+		<joint name="arm_joint_01">
 			<hardwareInterface>hardware_interface/EffortJointInterface</hardwareInterface>
 		</joint>
@@ -234,20 +225,10 @@
 		</actuator>
 	</transmission>
-	<transmission name="arm_joint_01_trans">
+	<transmission name="arm_joint_02_trans">
 		<type>transmission_interface/SimpleTransmission</type>
-		<joint name="arm_joint_01">
+		<joint name="arm_joint_02">
 			<hardwareInterface>hardware_interface/EffortJointInterface</hardwareInterface>
 		</joint>
 		<actuator name="motor2">
-			<hardwareInterface>hardware_interface/EffortJointInterface</hardwareInterface>
-			<mechanicalInterface>1</mechanicalInterface>
-		</actuator>
-	</transmission>
-	<transmission name="arm_joint_02_joint_trans">
-		<type>transmission_interface/SimpleTransmission</type>
-		<joint name="arm_joint_02">
-			<hardwareInterface>hardware_interface/EffortJointInterface</hardwareInterface>
-		</joint>
-		<actuator name="motor3">
 			<hardwareInterface>hardware_interface/EffortJointInterface</hardwareInterface>
 			<mechanicalInterface>1</mechanicalInterface>
@@ -259,5 +240,5 @@
 			<hardwareInterface>hardware_interface/EffortJointInterface</hardwareInterface>
 		</joint>
-		<actuator name="motor4">
+		<actuator name="motor3">
 			<hardwareInterface>hardware_interface/EffortJointInterface</hardwareInterface>
 			<mechanicalInterface>1</mechanicalInterface>

Commit message: position check to recharge

File: urdf/robot_assignment.xacro (robot description, xacro)
@@ -196,11 +196,11 @@
         <inertial>
             <origin xyz="0 0 0" rpy="0 0 0" />
-            <mass value="1" />
-            <xacro:cylinder_inertia mass="1" r="0.05" l="0.1" />
+            <mass value="1e-5" />
+            <xacro:box_inertia mass="1e-5" x="0.1" y="0.1" z="0.1"/>
         </inertial>
         <visual>
             <origin xyz="0 0 0" rpy="0 0 0" />
             <geometry>
-                <cylinder radius="0.05" length="0.1"/>
+                <box size="0.1 0.1 0.1"/>
             </geometry>
             <material name="blue" />
@@ -209,5 +209,5 @@
             <origin xyz="0 0 0" rpy="0 0 0"/>
             <geometry>
-                <cylinder radius="0.05" length="0.1"/>
+                <box size="0.1 0.1 0.1"/>
             </geometry>
         </collision>
